Commit message: xacro expansion

File: resources/bipanda/bipanda_spherized.urdf (robot description, URDF)
Before this commit: robot bipanda, 1 links, 0 joints
Links:
- added link left_panda_grasptarget, mass 0.0
- added link left_panda_hand, mass .81; collision sphere radius=0.024; collision sphere radius=0.024
- added link left_panda_leftfinger, mass 0.1; collision sphere radius=0.012; collision sphere radius=0.012
- added link left_panda_link0, mass 2.9; collision sphere radius=0.08; visual mesh filename=meshes/collision/link0.obj
- added link left_panda_link1, mass 2.7; collision sphere radius=0.06; collision sphere radius=0.06
- added link left_panda_link2, mass 2.73; collision sphere radius=0.06; collision sphere radius=0.06
- added link left_panda_link3, mass 2.04; collision sphere radius=0.05; collision sphere radius=0.055
- added link left_panda_link4, mass 2.08; collision sphere radius=0.055; collision sphere radius=0.055
- added link left_panda_link5, mass 3; collision sphere radius=0.025; collision sphere radius=0.025
- added link left_panda_link6, mass 1.3; collision sphere radius=0.05; collision sphere radius=0.05
- added link left_panda_link7, mass .2; collision sphere radius=0.02; collision sphere radius=0.02
- added link left_panda_link8, mass 0.0
- added link left_panda_rightfinger, mass 0.1; collision sphere radius=0.012; collision sphere radius=0.012
- added link right_panda_grasptarget, mass 0.0
- added link right_panda_hand, mass .81; collision sphere radius=0.024; collision sphere radius=0.024
- added link right_panda_leftfinger, mass 0.1; collision sphere radius=0.012; collision sphere radius=0.012
- added link right_panda_link0, mass 2.9; collision sphere radius=0.08; visual mesh filename=meshes/collision/link0.obj
- added link right_panda_link1, mass 2.7; collision sphere radius=0.06; collision sphere radius=0.06
- added link right_panda_link2, mass 2.73; collision sphere radius=0.06; collision sphere radius=0.06
- added link right_panda_link3, mass 2.04; collision sphere radius=0.05; collision sphere radius=0.055
- added link right_panda_link4, mass 2.08; collision sphere radius=0.055; collision sphere radius=0.055
- added link right_panda_link5, mass 3; collision sphere radius=0.025; collision sphere radius=0.025
- added link right_panda_link6, mass 1.3; collision sphere radius=0.05; collision sphere radius=0.05
- added link right_panda_link7, mass .2; collision sphere radius=0.02; collision sphere radius=0.02
- added link right_panda_link8, mass 0.0
- added link right_panda_rightfinger, mass 0.1; collision sphere radius=0.012; collision sphere radius=0.012
Joints:
- added joint left_mount: type fixed, parent world, child left_panda_link0, origin xyz=0 -0.2875 0 rpy=0 0 0
- added joint left_panda_finger_joint1: type fixed, parent left_panda_hand, child left_panda_leftfinger, origin xyz=0 0.065 0.0584 rpy=0 0 0, axis 0 1 0
- added joint left_panda_finger_joint2: type fixed, parent left_panda_hand, child left_panda_rightfinger, origin xyz=0 -0.065 0.0584 rpy=0 0 0, axis 0 -1 0, mimic joint=left_panda_finger_joint1
- added joint left_panda_grasptarget_hand: type fixed, parent left_panda_hand, child left_panda_grasptarget, origin xyz=0 0 0.105 rpy=0 0 0
- added joint left_panda_hand_joint: type fixed, parent left_panda_link8, child left_panda_hand, origin xyz=0 0 0 rpy=0 0 -0.785398163397
- added joint left_panda_joint1: type revolute, parent left_panda_link0, child left_panda_link1, origin xyz=0 0 0.333 rpy=0 0 0, axis 0 0 1, limit lower=-2.9671 upper=2.9671 effort=87 velocity=2.3925
- added joint left_panda_joint2: type revolute, parent left_panda_link1, child left_panda_link2, origin xyz=0 0 0 rpy=-1.57079632679 0 0, axis 0 0 1, limit lower=-1.8326 upper=1.8326 effort=87 velocity=2.3925
- added joint left_panda_joint3: type revolute, parent left_panda_link2, child left_panda_link3, origin xyz=0 -0.316 0 rpy=1.57079632679 0 0, axis 0 0 1, limit lower=-2.9671 upper=2.9671 effort=87 velocity=2.3925
- added joint left_panda_joint4: type revolute, parent left_panda_link3, child left_panda_link4, origin xyz=0.0825 0 0 rpy=1.57079632679 0 0, axis 0 0 1, limit lower=-3.1416 upper=0.0873 effort=87 velocity=2.3925
- added joint left_panda_joint5: type revolute, parent left_panda_link4, child left_panda_link5, origin xyz=-0.0825 0.384 0 rpy=-1.57079632679 0 0, axis 0 0 1, limit lower=-2.9671 upper=2.9671 effort=12 velocity=2.8710
- added joint left_panda_joint6: type revolute, parent left_panda_link5, child left_panda_link6, origin xyz=0 0 0 rpy=1.57079632679 0 0, axis 0 0 1, limit lower=-0.0873 upper=3.8223 effort=12 velocity=2.8710
- added joint left_panda_joint7: type revolute, parent left_panda_link6, child left_panda_link7, origin xyz=0.088 0 0 rpy=1.57079632679 0 0, axis 0 0 1, limit lower=-2.9671 upper=2.9671 effort=12 velocity=2.8710
- added joint left_panda_joint8: type fixed, parent left_panda_link7, child left_panda_link8, origin xyz=0 0 0.107 rpy=0 0 0, axis 0 0 0
- added joint right_mount: type fixed, parent world, child right_panda_link0, origin xyz=0 0.2875 0 rpy=0 0 0
- added joint right_panda_finger_joint1: type fixed, parent right_panda_hand, child right_panda_leftfinger, origin xyz=0 0.065 0.0584 rpy=0 0 0, axis 0 1 0
- added joint right_panda_finger_joint2: type fixed, parent right_panda_hand, child right_panda_rightfinger, origin xyz=0 -0.065 0.0584 rpy=0 0 0, axis 0 -1 0, mimic joint=right_panda_finger_joint1
- added joint right_panda_grasptarget_hand: type fixed, parent right_panda_hand, child right_panda_grasptarget, origin xyz=0 0 0.105 rpy=0 0 0
- added joint right_panda_hand_joint: type fixed, parent right_panda_link8, child right_panda_hand, origin xyz=0 0 0 rpy=0 0 -0.785398163397
- added joint right_panda_joint1: type revolute, parent right_panda_link0, child right_panda_link1, origin xyz=0 0 0.333 rpy=0 0 0, axis 0 0 1, limit lower=-2.9671 upper=2.9671 effort=87 velocity=2.3925
- added joint right_panda_joint2: type revolute, parent right_panda_link1, child right_panda_link2, origin xyz=0 0 0 rpy=-1.57079632679 0 0, axis 0 0 1, limit lower=-1.8326 upper=1.8326 effort=87 velocity=2.3925
- added joint right_panda_joint3: type revolute, parent right_panda_link2, child right_panda_link3, origin xyz=0 -0.316 0 rpy=1.57079632679 0 0, axis 0 0 1, limit lower=-2.9671 upper=2.9671 effort=87 velocity=2.3925
- added joint right_panda_joint4: type revolute, parent right_panda_link3, child right_panda_link4, origin xyz=0.0825 0 0 rpy=1.57079632679 0 0, axis 0 0 1, limit lower=-3.1416 upper=0.0873 effort=87 velocity=2.3925
- added joint right_panda_joint5: type revolute, parent right_panda_link4, child right_panda_link5, origin xyz=-0.0825 0.384 0 rpy=-1.57079632679 0 0, axis 0 0 1, limit lower=-2.9671 upper=2.9671 effort=12 velocity=2.8710
- added joint right_panda_joint6: type revolute, parent right_panda_link5, child right_panda_link6, origin xyz=0 0 0 rpy=1.57079632679 0 0, axis 0 0 1, limit lower=-0.0873 upper=3.8223 effort=12 velocity=2.8710
- added joint right_panda_joint7: type revolute, parent right_panda_link6, child right_panda_link7, origin xyz=0.088 0 0 rpy=1.57079632679 0 0, axis 0 0 1, limit lower=-2.9671 upper=2.9671 effort=12 velocity=2.8710
- added joint right_panda_joint8: type fixed, parent right_panda_link7, child right_panda_link8, origin xyz=0 0 0.107 rpy=0 0 0, axis 0 0 0

File: resources/bipanda/bipanda_spherized_1.urdf (robot description, URDF)
Before this commit: robot bipanda, 1 links, 0 joints
Links:
- added link left_panda_grasptarget, mass 0.0
- added link left_panda_hand, mass .81; collision sphere radius=0.104; visual mesh filename=meshes/visual/hand.obj
- added link left_panda_leftfinger, mass 0.1; collision sphere radius=0.024; visual mesh filename=meshes/visual/finger.obj
- added link left_panda_link0, mass 2.9; collision sphere radius=0.08; visual mesh filename=meshes/collision/link0.obj
- added link left_panda_link1, mass 2.7; collision sphere radius=0.154; visual mesh filename=meshes/visual/link1.obj
- added link left_panda_link2, mass 2.73; collision sphere radius=0.154; visual mesh filename=meshes/visual/link2.obj
- added link left_panda_link3, mass 2.04; collision sphere radius=0.128; visual mesh filename=meshes/visual/link3.obj
- added link left_panda_link4, mass 2.08; collision sphere radius=0.126; visual mesh filename=meshes/visual/link4.obj
- added link left_panda_link5, mass 3; collision sphere radius=0.176; visual mesh filename=meshes/visual/link5.obj
- added link left_panda_link6, mass 1.3; collision sphere radius=0.095; visual mesh filename=meshes/visual/link6.obj
- added link left_panda_link7, mass .2; collision sphere radius=0.072; visual mesh filename=meshes/collision/link7.obj
- added link left_panda_link8, mass 0.0
- added link left_panda_rightfinger, mass 0.1; collision sphere radius=0.024; visual mesh filename=meshes/visual/finger.obj
- added link right_panda_grasptarget, mass 0.0
- added link right_panda_hand, mass .81; collision sphere radius=0.104; visual mesh filename=meshes/visual/hand.obj
- added link right_panda_leftfinger, mass 0.1; collision sphere radius=0.024; visual mesh filename=meshes/visual/finger.obj
- added link right_panda_link0, mass 2.9; collision sphere radius=0.08; visual mesh filename=meshes/collision/link0.obj
- added link right_panda_link1, mass 2.7; collision sphere radius=0.154; visual mesh filename=meshes/visual/link1.obj
- added link right_panda_link2, mass 2.73; collision sphere radius=0.154; visual mesh filename=meshes/visual/link2.obj
- added link right_panda_link3, mass 2.04; collision sphere radius=0.128; visual mesh filename=meshes/visual/link3.obj
- added link right_panda_link4, mass 2.08; collision sphere radius=0.126; visual mesh filename=meshes/visual/link4.obj
- added link right_panda_link5, mass 3; collision sphere radius=0.176; visual mesh filename=meshes/visual/link5.obj
- added link right_panda_link6, mass 1.3; collision sphere radius=0.095; visual mesh filename=meshes/visual/link6.obj
- added link right_panda_link7, mass .2; collision sphere radius=0.072; visual mesh filename=meshes/collision/link7.obj
- added link right_panda_link8, mass 0.0
- added link right_panda_rightfinger, mass 0.1; collision sphere radius=0.024; visual mesh filename=meshes/visual/finger.obj
Joints:
- added joint left_mount: type fixed, parent world, child left_panda_link0, origin xyz=0 -0.2875 0 rpy=0 0 0
- added joint left_panda_finger_joint1: type fixed, parent left_panda_hand, child left_panda_leftfinger, origin xyz=0 0.065 0.0584 rpy=0 0 0, axis 0 1 0
- added joint left_panda_finger_joint2: type fixed, parent left_panda_hand, child left_panda_rightfinger, origin xyz=0 -0.065 0.0584 rpy=0 0 0, axis 0 -1 0, mimic joint=left_panda_finger_joint1
- added joint left_panda_grasptarget_hand: type fixed, parent left_panda_hand, child left_panda_grasptarget, origin xyz=0 0 0.105 rpy=0 0 0
- added joint left_panda_hand_joint: type fixed, parent left_panda_link8, child left_panda_hand, origin xyz=0 0 0 rpy=0 0 -0.785398163397
- added joint left_panda_joint1: type revolute, parent left_panda_link0, child left_panda_link1, origin xyz=0 0 0.333 rpy=0 0 0, axis 0 0 1, limit lower=-2.9671 upper=2.9671 effort=87 velocity=2.3925
- added joint left_panda_joint2: type revolute, parent left_panda_link1, child left_panda_link2, origin xyz=0 0 0 rpy=-1.57079632679 0 0, axis 0 0 1, limit lower=-1.8326 upper=1.8326 effort=87 velocity=2.3925
- added joint left_panda_joint3: type revolute, parent left_panda_link2, child left_panda_link3, origin xyz=0 -0.316 0 rpy=1.57079632679 0 0, axis 0 0 1, limit lower=-2.9671 upper=2.9671 effort=87 velocity=2.3925
- added joint left_panda_joint4: type revolute, parent left_panda_link3, child left_panda_link4, origin xyz=0.0825 0 0 rpy=1.57079632679 0 0, axis 0 0 1, limit lower=-3.1416 upper=0.0873 effort=87 velocity=2.3925
- added joint left_panda_joint5: type revolute, parent left_panda_link4, child left_panda_link5, origin xyz=-0.0825 0.384 0 rpy=-1.57079632679 0 0, axis 0 0 1, limit lower=-2.9671 upper=2.9671 effort=12 velocity=2.8710
- added joint left_panda_joint6: type revolute, parent left_panda_link5, child left_panda_link6, origin xyz=0 0 0 rpy=1.57079632679 0 0, axis 0 0 1, limit lower=-0.0873 upper=3.8223 effort=12 velocity=2.8710
- added joint left_panda_joint7: type revolute, parent left_panda_link6, child left_panda_link7, origin xyz=0.088 0 0 rpy=1.57079632679 0 0, axis 0 0 1, limit lower=-2.9671 upper=2.9671 effort=12 velocity=2.8710
- added joint left_panda_joint8: type fixed, parent left_panda_link7, child left_panda_link8, origin xyz=0 0 0.107 rpy=0 0 0, axis 0 0 0
- added joint right_mount: type fixed, parent world, child right_panda_link0, origin xyz=0 0.2875 0 rpy=0 0 0
- added joint right_panda_finger_joint1: type fixed, parent right_panda_hand, child right_panda_leftfinger, origin xyz=0 0.065 0.0584 rpy=0 0 0, axis 0 1 0
- added joint right_panda_finger_joint2: type fixed, parent right_panda_hand, child right_panda_rightfinger, origin xyz=0 -0.065 0.0584 rpy=0 0 0, axis 0 -1 0, mimic joint=right_panda_finger_joint1
- added joint right_panda_grasptarget_hand: type fixed, parent right_panda_hand, child right_panda_grasptarget, origin xyz=0 0 0.105 rpy=0 0 0
- added joint right_panda_hand_joint: type fixed, parent right_panda_link8, child right_panda_hand, origin xyz=0 0 0 rpy=0 0 -0.785398163397
- added joint right_panda_joint1: type revolute, parent right_panda_link0, child right_panda_link1, origin xyz=0 0 0.333 rpy=0 0 0, axis 0 0 1, limit lower=-2.9671 upper=2.9671 effort=87 velocity=2.3925
- added joint right_panda_joint2: type revolute, parent right_panda_link1, child right_panda_link2, origin xyz=0 0 0 rpy=-1.57079632679 0 0, axis 0 0 1, limit lower=-1.8326 upper=1.8326 effort=87 velocity=2.3925
- added joint right_panda_joint3: type revolute, parent right_panda_link2, child right_panda_link3, origin xyz=0 -0.316 0 rpy=1.57079632679 0 0, axis 0 0 1, limit lower=-2.9671 upper=2.9671 effort=87 velocity=2.3925
- added joint right_panda_joint4: type revolute, parent right_panda_link3, child right_panda_link4, origin xyz=0.0825 0 0 rpy=1.57079632679 0 0, axis 0 0 1, limit lower=-3.1416 upper=0.0873 effort=87 velocity=2.3925
- added joint right_panda_joint5: type revolute, parent right_panda_link4, child right_panda_link5, origin xyz=-0.0825 0.384 0 rpy=-1.57079632679 0 0, axis 0 0 1, limit lower=-2.9671 upper=2.9671 effort=12 velocity=2.8710
- added joint right_panda_joint6: type revolute, parent right_panda_link5, child right_panda_link6, origin xyz=0 0 0 rpy=1.57079632679 0 0, axis 0 0 1, limit lower=-0.0873 upper=3.8223 effort=12 velocity=2.8710
- added joint right_panda_joint7: type revolute, parent right_panda_link6, child right_panda_link7, origin xyz=0.088 0 0 rpy=1.57079632679 0 0, axis 0 0 1, limit lower=-2.9671 upper=2.9671 effort=12 velocity=2.8710
- added joint right_panda_joint8: type fixed, parent right_panda_link7, child right_panda_link8, origin xyz=0 0 0.107 rpy=0 0 0, axis 0 0 0
