Commit message: fix link 5 torch

File: resources/m900ib/spherized.urdf (robot description, URDF)
Before this commit: robot fanuc_m900ib700l, 13 links, 12 joints
Links:
- link base_link: geometry collision sphere radius=0.347906; collision sphere radius=0.355754
- link link_1: geometry collision sphere radius=0.452197; collision sphere radius=0.464921
