Commit message: adding flyer

File: resources/g1_description/spherized.urdf (robot description, URDF)
Before this commit: robot g1_29dof, 40 links, 39 joints
Links:
- added link left_foot, mass 0.0
- added link right_foot, mass 0.0
- link left_ankle_roll_link: geometry collision sphere radius=0.025; collision sphere radius=0.025
- link right_ankle_roll_link: geometry collision sphere radius=0.025; collision sphere radius=0.025
Joints:
- added joint left_foot_joint: type fixed, parent left_ankle_roll_link, child left_foot, origin xyz=0.1 0 0 rpy=0 0 0
- added joint right_foot_joint: type fixed, parent right_ankle_roll_link, child right_foot, origin xyz=0.1 0 0 rpy=0 0 0

Commit message: add se3 ops and add a self collision constraint

File: resources/g1_description/spherized.urdf (robot description, URDF)
Before this commit: robot g1_29dof, 42 links, 41 joints
Links:
- added link floating_pitch
- added link floating_roll
- added link floating_x
- added link floating_y
- added link floating_yaw
- added link floating_z
- added link world
Joints:
- added joint pitch_to_yaw: type revolute, parent floating_pitch, child floating_yaw, axis 0 0 1, limit lower=-3.14159 upper=3.14159 effort=0 velocity=0
- added joint roll_to_pitch: type revolute, parent floating_roll, child floating_pitch, axis 0 1 0, limit lower=-3.14159 upper=3.14159 effort=0 velocity=0
- added joint world_to_x: type prismatic, parent world, child floating_x, axis 1 0 0, limit lower=-2.0 upper=2.0 effort=0 velocity=0
- added joint x_to_y: type prismatic, parent floating_x, child floating_y, axis 0 1 0, limit lower=-2.0 upper=2.0 effort=0 velocity=0
- added joint y_to_z: type prismatic, parent floating_y, child floating_z, axis 0 0 1, limit lower=-2.0 upper=2.0 effort=0 velocity=0
- added joint yaw_to_pelvis: type fixed, parent floating_yaw, child pelvis
- added joint z_to_roll: type revolute, parent floating_z, child floating_roll, axis 1 0 0, limit lower=-3.14159 upper=3.14159 effort=0 velocity=0
