Commit message: fetch

File: resources/fetch/fetch_spherized.urdf (robot description, URDF)
Before this commit: robot fetch, 17 links, 16 joints
Links:
- link base_link: mass None -> 70.1294
- link bellows_link: mass None -> 0.169374038216602
- link elbow_flex_link: mass None -> 2.1299
- link forearm_roll_link: mass None -> 1.6563
- link gripper_link: mass None -> 1.5175
- link head_pan_link: mass None -> 2.2556
- link head_tilt_link: mass None -> 0.9087
- link l_gripper_finger_link: mass None -> 0.0798
- link r_gripper_finger_link: mass None -> 0.0798
- link shoulder_lift_link: mass None -> 2.6615
- link shoulder_pan_link: mass None -> 2.5587
- link torso_fixed_link: mass None -> 13.2775
- link torso_lift_link: mass None -> 10.7796
- link upperarm_roll_link: mass None -> 2.3311
- link wrist_flex_link: mass None -> 1.725
- link wrist_roll_link: mass None -> 0.1354
