Commit message: base version works

File: resources/iiwa_marker/iiwa_marker_spherized.urdf (robot description, URDF)
Before this commit: robot iiwa, 16 links, 15 joints
Links:
- removed link panda_marker
- removed link panda_marker_holder
- removed link panda_tip
- added link iiwa_marker, mass 0.05; collision sphere radius=0.007140500005334616; collision sphere radius=0.007258803583681583
- added link iiwa_marker_holder, mass 0.2; collision sphere radius=0.0156889446079731; collision sphere radius=0.016278699040412903
- added link iiwa_tip, mass 0.01; collision sphere radius=0.000999373965896666; collision sphere radius=0.000999373965896666
Joints:
- removed joint panda_marker_holder_joint
- removed joint panda_marker_joint
- removed joint panda_tip_joint
- added joint iiwa_marker_holder_joint: type fixed, parent marker_attach, child iiwa_marker_holder, origin xyz=-0.01 -0.032 0.065 rpy=0 0 0
- added joint iiwa_marker_joint: type fixed, parent iiwa_marker_holder, child iiwa_marker, origin xyz=-0.075 0.0285 0.15 rpy=-1.57079632679 0 0
- added joint iiwa_tip_joint: type fixed, parent iiwa_marker, child iiwa_tip, origin xyz=0.08125 0.0035 0.003625 rpy=0 0 0

Commit message: fk doesnt work perfect rest are good, se3 is now 8 to account for self-motion-manifold param

File: resources/iiwa_marker/iiwa_marker_spherized.urdf (robot description, URDF)
Before this commit: robot iiwa, 16 links, 15 joints
Links:
- added link iiwa_frame_link_ee
Joints:
- added joint iiwa_frame_ee_joint: type fixed, parent iiwa_link_ee, child iiwa_frame_link_ee, origin xyz=0.09 0 0 rpy=3.141592653589793 0 1.570796326794897

Commit message: maze for iiwa works

File: resources/iiwa_marker/iiwa_marker_spherized.urdf (robot description, URDF)
Before this commit: robot iiwa, 17 links, 16 joints
Links:
- removed link iiwa_frame_link_ee
- link iiwa_link_0: geometry collision sphere radius=0.10320371389389038; collision sphere radius=0.1034880056977272
- link iiwa_link_1: geometry collision sphere radius=0.07707267999649048; collision sphere radius=0.07754990458488464
- link iiwa_link_2: geometry collision sphere radius=0.07557239383459091; collision sphere radius=0.07711803913116455
- link iiwa_link_3: geometry collision sphere radius=0.06575722992420197; collision sphere radius=0.06575722992420197
- link iiwa_link_4: geometry collision sphere radius=0.0663609728217125; collision sphere radius=0.06794817000627518
- link iiwa_link_5: geometry collision sphere radius=0.04509371891617775; collision sphere radius=0.04663007706403732
- link iiwa_link_6: geometry collision sphere radius=0.06905970722436905; collision sphere radius=0.07132092118263245
- link iiwa_link_7: geometry collision sphere radius=0.02980879507958889; collision sphere radius=0.02980879507958889
- link iiwa_marker: geometry collision sphere radius=0.005364664364606142; collision sphere radius=0.005398083943873644
- link iiwa_marker_holder: geometry collision sphere radius=0.015679605305194855; collision sphere radius=0.01659444347023964
- link iiwa_tip: geometry collision sphere radius=0.0010131720919162035; collision sphere radius=0.0010209220927208662
Joints:
- removed joint iiwa_frame_ee_joint
